Commit message: simulation coming together

File: gt_car_vehicle_description/urdf/gt_car.urdf.xacro (robot description, xacro)
@@ -345,7 +345,4 @@
     </inertial>
   </link>
- <!--  <gazebo reference="laser_box">
-    <material>Gazebo/Green</material>
-  </gazebo> -->
   <joint name="laser_joint" type="fixed">
     <origin xyz="0 0 0.07" rpy="0 0 0" />
@@ -353,4 +350,26 @@
     <child link="laser_box" />
   </joint>
+ <link name="camera_box">
+    <visual>
+      <origin xyz="-0.015 0 0" rpy="0 0 0" />
+      <geometry>
+	<box size="0.015 0.05 0.04"/>
+      </geometry>
+      <material name="black"/>
+    </visual>
+    <inertial>
+      <mass value="0.001"/>
+      <origin xyz="0 0 0"/>
+      <inertia ixx="0.0001" ixy="0.0" ixz="0.0" iyy="0.0001" iyz="0.0" izz="0.0001"/>
+    </inertial>
+  </link>
+  <joint name="camera_joint" type="fixed">
+    <origin xyz="0.15 0 0.02" rpy="0 0 0" />
+    <parent link="layer_2" />
+    <child link="camera_box" />
+  </joint>
+  <gazebo reference="camera_box">
+    <material>Gazebo/Black</material>
+  </gazebo>
  <gazebo reference="laser_box">
     <sensor type="ray" name="head_hokuyo_sensor">
@@ -361,19 +380,19 @@
         <scan>
           <horizontal>
-            <samples>720</samples>
+            <samples>1080</samples>
             <resolution>1</resolution>
-            <min_angle>-1.570796</min_angle>
-            <max_angle>1.570796</max_angle>
+            <min_angle>-2.35619449</min_angle>
+            <max_angle>2.35619449</max_angle>
           </horizontal>
         </scan>
         <range>
-          <min>0.10</min>
-          <max>30.0</max>
-          <resolution>0.01</resolution>
+          <min>0.04</min>
+          <max>10.0</max>
+          <resolution>0.001</resolution>
         </range>
         <noise>
           <type>gaussian</type>
           <mean>0.0</mean>
-          <stddev>0.01</stddev>
+          <stddev>0.013</stddev>
         </noise>
       </ray>
@@ -384,4 +403,45 @@
     </sensor>
   </gazebo>
+ <!-- camera -->
+  <gazebo reference="camera_box">
+    <material name="Black"/>
+    <sensor type="camera" name="camera1">
+      <update_rate>30.0</update_rate>
+      <camera name="head">
+        <horizontal_fov>1.3962634</horizontal_fov>
+        <image>
+          <width>800</width>
+          <height>800</height>
+          <format>R8G8B8</format>
+        </image>
+        <clip>
+          <near>0.02</near>
+          <far>300</far>
+        </clip>
+        <noise>
+          <type>gaussian</type>
+          <!-- Noise is sampled independently per pixel on each frame.
+               That pixel's noise value is added to each of its color
+               channels, which at that point lie in the range [0,1]. -->
+          <mean>0.0</mean>
+          <stddev>0.007</stddev>
+        </noise>
+      </camera>
+      <plugin name="camera_controller" filename="libgazebo_ros_camera.so">
+        <alwaysOn>true</alwaysOn>
+        <updateRate>0.0</updateRate>
+        <cameraName>camera1</cameraName>
+        <imageTopicName>image_raw</imageTopicName>
+        <cameraInfoTopicName>camera_info</cameraInfoTopicName>
+        <frameName>camera_box</frameName>
+        <hackBaseline>0.07</hackBaseline>
+        <distortionK1>0.0</distortionK1>
+        <distortionK2>0.0</distortionK2>
+        <distortionK3>0.0</distortionK3>
+        <distortionT1>0.0</distortionT1>
+        <distortionT2>0.0</distortionT2>
+      </plugin>
+    </sensor>
+  </gazebo>
   <gazebo>
     <plugin name="gazebo_ros_control" filename="libgazebo_ros_control.so"/>

Commit message: Added validation boolean in tracker to prevent turn around if rolling out of threshold changed dimension to be more similar to the actual car

File: gt_car_vehicle_description/urdf/gt_car.urdf.xacro (robot description, xacro)
@@ -27,6 +27,6 @@
        from a U joint to the corresponding hex hub. wheel_travel is the
        vertical wheel travel. -->
-  <xacro:property name="wheelbase" value="0.335"/>
-  <xacro:property name="hex_hub_dist" value="0.265"/>
+  <xacro:property name="wheelbase" value="0.325"/>
+  <xacro:property name="hex_hub_dist" value="0.285"/>
   <xacro:property name="axle_length" value="0.00"/>
   <xacro:property name="wheel_travel" value="0.04"/>
@@ -288,5 +288,5 @@
   </gazebo>
   <joint name="chassis_to_layer_1" type="fixed">
-    <origin xyz="0 0 0.05" rpy="0 0 0" />
+    <origin xyz="0 0 0.075" rpy="0 0 0" />
     <parent link="chassis"/>
     <child link="layer_1"/>
@@ -317,5 +317,5 @@
   </gazebo>
   <joint name="chassis_to_layer_2" type="fixed">
-    <origin xyz="0 0 0.1" rpy="0 0 0" />
+    <origin xyz="0 0 0.115" rpy="0 0 0" />
     <parent link="chassis"/>
     <child link="layer_2"/>

Commit message: tuning and debugging

File: gt_car_vehicle_description/urdf/gt_car.urdf.xacro (robot description, xacro)
@@ -22,5 +22,5 @@
   <xacro:property name="tire_width" value="0.05"/>
   <xacro:property name="hex_hub_depth" value="0.025"/>
-  <xacro:property name="wheel_mass" value="0.2"/>
+  <xacro:property name="wheel_mass" value="0.5"/>
   <!-- hex_hub_dist is the distance between left and right hex hubs when
        the shock absorbers are fully extended. axle_length is the distance
@@ -173,4 +173,14 @@
           <cylinder radius="${tire_dia / 2}" length="${tire_width}"/>
         </geometry>
+	<surface>
+          <friction>
+            <ode>
+              <mu>10.0</mu>
+              <mu2>10.0</mu2>
+              <slip1>0.0</slip1>
+              <slip2>0.0</slip2>
+            </ode>
+          </friction>
+        </surface>
       </collision>
       <xacro:thick_walled_tube_inertial
